Commit message: Fix urdf and config.

File: manipulator_assets/swing_arm/description/urdf/arm.urdf.xacro (robot description, xacro)
@@ -23,13 +23,14 @@
                        iyy="2226000" iyz="1036.356" izz="2291000"
                        mesh_file="package://swing_arm/description/meshes/link3.stl" material_name="silver"
-                       inertial_xyz="0.191296 -0.001405 0.053882"/>
-    <xacro:create_link name="link4" mass="0.056678"
+                       inertial_xyz="0.191296 -0.001405 0.053882"
+                       collision_scale_y="0.8"/>
+    <xacro:create_link name="link4" mass="0.1"
                        ixx="1262.246" ixy="32.61" ixz="-553.334"
-                       iyy="1346.829" iyz="41.18" izz="975.984"
+                       iyy="100000" iyz="41.18" izz="975.984"
                        mesh_file="package://swing_arm/description/meshes/link4.stl" material_name="silver"
                        inertial_xyz="0.02969 0.00192 0.03765"/>
     <xacro:create_link name="link5" mass="0.598593"
                        ixx="735400" ixy="-449.048" ixz="37386.443"
-                       iyy="732800" iyz="-210.043" izz="238600"
+                       iyy="732800" iyz="-210.043" izz="500000"
                        mesh_file="package://swing_arm/description/meshes/link5.stl" material_name="silver"
                        inertial_xyz="0.001992 -0.000088 -0.053421"/>

File: manipulator_common/include/manipulator_common/utilities/urdf/common.xacro (robot description, xacro)
@@ -1,7 +1,6 @@
 <?xml version="1.0"?>
 <robot xmlns:xacro="http://ros.org/wiki/xacro">
-    <xacro:property name="scale_factor" value="1e-9"/>
     <!-- Macro for creating links -->
-    <xacro:macro name="create_link" params="name mass ixx ixy ixz iyy iyz izz mesh_file material_name inertial_xyz='0 0 0'">
+    <xacro:macro name="create_link" params="name mass ixx ixy ixz iyy iyz izz mesh_file material_name collision_file:=none scale_factor:=1e-9 collision_scale_x:=1 collision_scale_y:=1 collision_scale_z:=1 inertial_xyz:='0 0 0'">
         <link name="${name}">
             <inertial>
@@ -21,5 +20,10 @@
                 <origin xyz="0 0 0" rpy="0 0 0"/>
                 <geometry>
-                    <mesh filename="${mesh_file}"/>
+                    <xacro:if value="${collision_file == 'none'}">
+                        <mesh filename="${mesh_file}" scale="${collision_scale_x} ${collision_scale_y} ${collision_scale_z}"/>
+                    </xacro:if>
+                    <xacro:unless value="${collision_file == 'none'}">
+                        <mesh filename="${collision_file}" scale="${collision_scale_x} ${collision_scale_y} ${collision_scale_z}"/>
+                    </xacro:unless>
                 </geometry>
             </collision>
