Commit message: Add gripper assets.

File: manipulator_common/include/manipulator_common/utilities/urdf/common.xacro (robot description, xacro)
@@ -42,4 +42,8 @@
                 <limit lower="${lower}" upper="${upper}" effort="${effort}" velocity="${velocity}"/>
             </xacro:if>
+            <xacro:if value="${type == 'prismatic'}">
+                <axis xyz="${axis_xyz}"/>
+                <limit lower="${lower}" upper="${upper}" effort="${effort}" velocity="${velocity}"/>
+            </xacro:if>
         </joint>
     </xacro:macro>

Commit message: Add urdf temple rpy.

File: manipulator_common/include/manipulator_common/utilities/urdf/common.xacro (robot description, xacro)
@@ -5,8 +5,8 @@
                  params="name mass ixx ixy ixz iyy iyz izz mesh_file collision_file:=none scale_factor:=1e-9
                         collision_scale_x:=1 collision_scale_y:=1 collision_scale_z:=1
-                        vision_scales:='1 1 1' inertial_xyz:='0 0 0'">
+                        vision_scales:='1 1 1' inertial_xyz:='0 0 0' xyz:='0 0 0' rpy:='0 0 0'">
         <link name="${name}">
             <inertial>
-                <origin xyz="${inertial_xyz}" rpy="0 0 0"/>
+                <origin xyz="${inertial_xyz}" rpy="${rpy}"/>
                 <mass value="${mass}"/>
                 <inertia ixx="${ixx * scale_factor}" ixy="${ixy * scale_factor}" ixz="${ixz * scale_factor}"
@@ -14,5 +14,5 @@
             </inertial>
             <visual>
-                <origin xyz="0 0 0" rpy="0 0 0"/>
+                <origin xyz="${xyz}" rpy="${rpy}"/>
                 <geometry>
                     <mesh filename="${mesh_file}"
@@ -21,5 +21,5 @@
             </visual>
             <collision>
-                <origin xyz="0 0 0" rpy="0 0 0"/>
+                <origin xyz="${xyz}" rpy="${rpy}"/>
                 <geometry>
                     <xacro:if value="${collision_file == 'none'}">
